File: pcb/EOL/EOL.kicad_sch (KiCad schematic)
At the start: 16 parts

Commit message: Update sch.
Parts:
- H1, H2, H3, H4: value (none) -> MountingHole; footprint (none) -> MountingHole:MountingHole_3.2mm_M3_Pad_Via
- J1: value (none) -> Conn_01x06; footprint (none) -> External:PHOENIX_1985234
- R1, R3, R4: value (none) -> 2k; footprint (none) -> Resistor_SMD:R_0603_1608Metric_Pad1.05x0.95mm_HandSolder
- R2: value (none) -> 1k; footprint (none) -> Resistor_SMD:R_0603_1608Metric_Pad1.05x0.95mm_HandSolder
- SW1, SW2, SW3, SW4: value (none) -> Slide_DPDT; footprint (none) -> Button_Switch_THT:SW_E-Switch_EG1271_DPDT
- SW5, SW6, SW7: value (none) -> SW_Push_DPDT; footprint (none) -> External:MHPS2285
Changed lines of the file:
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@@
     (in_bom yes) (on_board yes)
     (property "Reference" "R3" (id 0) (at 86.36 41.7322 90))
-    (property "Value" "" (id 1) (at 86.36 44.0436 90))
-    (property "Footprint" "" (id 2) (at 86.36 45.212 90)
+    (property "Value" "2k" (id 1) (at 86.36 44.0436 90))
+    (property "Footprint" "Resistor_SMD:R_0603_1608Metric_Pad1.05x0.95mm_HandSolder" (id 2) (at 86.36 45.212 90)
       (effects (font (size 1.27 1.27)) hide)
     )
@@
       (effects (font (size 1.27 1.27)) (justify right))
     )
-    (property "Value" "" (id 1) (at 71.628 101.473 0)
-      (effects (font (size 1.27 1.27)) (justify right))
-    )
-    (property "Footprint" "" (id 2) (at 71.628 100.33 90)
+    (property "Value" "2k" (id 1) (at 71.628 101.473 0)
+      (effects (font (size 1.27 1.27)) (justify right))
+    )
+    (property "Footprint" "Resistor_SMD:R_0603_1608Metric_Pad1.05x0.95mm_HandSolder" (id 2) (at 71.628 100.33 90)
       (effects (font (size 1.27 1.27)) hide)
     )
@@
     (in_bom yes) (on_board yes)
     (property "Reference" "SW7" (id 0) (at 100.33 39.751 0))
-    (property "Value" "" (id 1) (at 100.33 42.0624 0))
-    (property "Footprint" "" (id 2) (at 100.33 46.99 0)
+    (property "Value" "SW_Push_DPDT" (id 1) (at 100.33 42.0624 0))
+    (property "Footprint" "External:MHPS2285" (id 2) (at 100.33 46.99 0)
       (effects (font (size 1.27 1.27)) hide)
     )
@@
     (in_bom yes) (on_board yes)
     (property "Reference" "SW3" (id 0) (at 68.58 42.291 0))
-    (property "Value" "" (id 1) (at 68.58 44.6024 0))
-    (property "Footprint" "" (id 2) (at 68.58 49.53 0)
+    (property "Value" "Slide_DPDT" (id 1) (at 68.58 44.6024 0))
+    (property "Footprint" "Button_Switch_THT:SW_E-Switch_EG1271_DPDT" (id 2) (at 68.58 49.53 0)
       (effects (font (size 1.27 1.27)) hide)
     )
@@
       (effects (font (size 1.27 1.27)) (justify left))
     )
-    (property "Value" "" (id 1) (at 165.1 87.503 0)
-      (effects (font (size 1.27 1.27)) (justify left))
-    )
-    (property "Footprint" "" (id 2) (at 162.56 86.36 0)
+    (property "Value" "MountingHole" (id 1) (at 165.1 87.503 0)
+      (effects (font (size 1.27 1.27)) (justify left))
+    )
+    (property "Footprint" "MountingHole:MountingHole_3.2mm_M3_Pad_Via" (id 2) (at 162.56 86.36 0)
       (effects (font (size 1.27 1.27)) hide)
     )
@@
       (effects (font (size 1.27 1.27)) (justify left))
     )
-    (property "Value" "" (id 1) (at 185.42 87.503 0)
-      (effects (font (size 1.27 1.27)) (justify left))
-    )
-    (property "Footprint" "" (id 2) (at 182.88 86.36 0)
+    (property "Value" "MountingHole" (id 1) (at 185.42 87.503 0)
+      (effects (font (size 1.27 1.27)) (justify left))
+    )
+    (property "Footprint" "MountingHole:MountingHole_3.2mm_M3_Pad_Via" (id 2) (at 182.88 86.36 0)
       (effects (font (size 1.27 1.27)) hide)
     )
@@
       (effects (font (size 1.27 1.27)) (justify left))
     )
-    (property "Value" "" (id 1) (at 165.1 95.123 0)
-      (effects (font (size 1.27 1.27)) (justify left))
-    )
-    (property "Footprint" "" (id 2) (at 162.56 93.98 0)
+    (property "Value" "MountingHole" (id 1) (at 165.1 95.123 0)
+      (effects (font (size 1.27 1.27)) (justify left))
+    )
+    (property "Footprint" "MountingHole:MountingHole_3.2mm_M3_Pad_Via" (id 2) (at 162.56 93.98 0)
       (effects (font (size 1.27 1.27)) hide)
     )
@@
       (effects (font (size 1.27 1.27)) (justify left))
     )
-    (property "Value" "" (id 1) (at 185.42 95.123 0)
-      (effects (font (size 1.27 1.27)) (justify left))
-    )
-    (property "Footprint" "" (id 2) (at 182.88 93.98 0)
+    (property "Value" "MountingHole" (id 1) (at 185.42 95.123 0)
+      (effects (font (size 1.27 1.27)) (justify left))
+    )
+    (property "Footprint" "MountingHole:MountingHole_3.2mm_M3_Pad_Via" (id 2) (at 182.88 93.98 0)
       (effects (font (size 1.27 1.27)) hide)
     )
@@
     (in_bom yes) (on_board yes)
     (property "Reference" "SW1" (id 0) (at 57.15 100.965 0))
-    (property "Value" "" (id 1) (at 57.15 103.2764 0))
-    (property "Footprint" "" (id 2) (at 57.15 119.38 0)
+    (property "Value" "Slide_DPDT" (id 1) (at 57.15 103.2764 0))
+    (property "Footprint" "Button_Switch_THT:SW_E-Switch_EG1271_DPDT" (id 2) (at 57.15 119.38 0)
       (effects (font (size 1.27 1.27)) hide)
     )
@@
     (in_bom yes) (on_board yes)
     (property "Reference" "SW5" (id 0) (at 82.55 84.201 0))
-    (property "Value" "" (id 1) (at 82.55 86.5124 0))
-    (property "Footprint" "" (id 2) (at 82.55 91.44 0)
+    (property "Value" "SW_Push_DPDT" (id 1) (at 82.55 86.5124 0))
+    (property "Footprint" "External:MHPS2285" (id 2) (at 82.55 91.44 0)
       (effects (font (size 1.27 1.27)) hide)
     )
@@
       (effects (font (size 1.27 1.27)) (justify right))
     )
-    (property "Value" "" (id 1) (at 88.138 154.813 0)
-      (effects (font (size 1.27 1.27)) (justify right))
-    )
-    (property "Footprint" "" (id 2) (at 88.138 153.67 90)
+    (property "Value" "2k" (id 1) (at 88.138 154.813 0)
+      (effects (font (size 1.27 1.27)) (justify right))
+    )
+    (property "Footprint" "Resistor_SMD:R_0603_1608Metric_Pad1.05x0.95mm_HandSolder" (id 2) (at 88.138 153.67 90)
       (effects (font (size 1.27 1.27)) hide)
     )
@@
     (in_bom yes) (on_board yes)
     (property "Reference" "SW4" (id 0) (at 73.66 164.465 0))
-    (property "Value" "" (id 1) (at 73.66 166.7764 0))
-    (property "Footprint" "" (id 2) (at 73.66 182.88 0)
+    (property "Value" "Slide_DPDT" (id 1) (at 73.66 166.7764 0))
+    (property "Footprint" "Button_Switch_THT:SW_E-Switch_EG1271_DPDT" (id 2) (at 73.66 182.88 0)
       (effects (font (size 1.27 1.27)) hide)
     )
@@
     (in_bom yes) (on_board yes)
     (property "Reference" "SW6" (id 0) (at 99.06 137.541 0))
-    (property "Value" "" (id 1) (at 99.06 139.8524 0))
-    (property "Footprint" "" (id 2) (at 99.06 144.78 0)
+    (property "Value" "SW_Push_DPDT" (id 1) (at 99.06 139.8524 0))
+    (property "Footprint" "External:MHPS2285" (id 2) (at 99.06 144.78 0)
       (effects (font (size 1.27 1.27)) hide)
     )
@@
     (in_bom yes) (on_board yes)
     (property "Reference" "R2" (id 0) (at 78.74 139.5222 90))
-    (property "Value" "" (id 1) (at 78.74 141.8336 90))
-    (property "Footprint" "" (id 2) (at 78.74 143.002 90)
+    (property "Value" "1k" (id 1) (at 78.74 141.8336 90))
+    (property "Footprint" "Resistor_SMD:R_0603_1608Metric_Pad1.05x0.95mm_HandSolder" (id 2) (at 78.74 143.002 90)
       (effects (font (size 1.27 1.27)) hide)
     )
@@
     (in_bom yes) (on_board yes)
     (property "Reference" "SW2" (id 0) (at 66.04 140.081 0))
-    (property "Value" "" (id 1) (at 66.04 142.3924 0))
-    (property "Footprint" "" (id 2) (at 66.04 147.32 0)
+    (property "Value" "Slide_DPDT" (id 1) (at 66.04 142.3924 0))
+    (property "Footprint" "Button_Switch_THT:SW_E-Switch_EG1271_DPDT" (id 2) (at 66.04 147.32 0)
       (effects (font (size 1.27 1.27)) hide)
     )
@@
       (effects (font (size 1.27 1.27)) (justify left))
     )
-    (property "Value" "" (id 1) (at 160.528 65.2022 0)
-      (effects (font (size 1.27 1.27)) (justify left))
-    )
-    (property "Footprint" "" (id 2) (at 162.56 62.23 0)
+    (property "Value" "Conn_01x06" (id 1) (at 160.528 65.2022 0)
+      (effects (font (size 1.27 1.27)) (justify left))
+    )
+    (property "Footprint" "External:PHOENIX_1985234" (id 2) (at 162.56 62.23 0)
       (effects (font (size 1.27 1.27)) hide)
     )
@@
     )
     (path "/e41566cb-430e-47cc-a443-f9429357a050"
-      (reference "J1") (unit 1) (value "Conn_01x06") (footprint "")
+      (reference "J1") (unit 1) (value "Conn_01x06") (footprint "External:PHOENIX_1985234")
     )
     (path "/00000000-0000-0000-0000-00006235fba3"

Commit message: Replace the terminal footprint for a screw terminal. Added the LCSC unique ids to ease the process of ordering a pcb.
Parts:
- J1: footprint External:PHOENIX_1985234 -> TerminalBlock_Phoenix:TerminalBlock_Phoenix_MKDS-1,5-6_1x06_P5.00mm_Horizontal; LCSC (none) -> C2802619
- R1, R3: value 2k -> 2k2; LCSC (none) -> C5140136
- R2: value 1k -> 2k2; LCSC (none) -> C5140136
- R4: value 2k -> 1k; LCSC (none) -> C3152127
- SW1, SW2, SW3, SW4: LCSC (none) -> C2906278
- SW5, SW6, SW7: LCSC (none) -> C493261
Connections:
- net DL: now also J1.2 (Pin_2); no longer J1.5 (Pin_5)
- net IN1: now also J1.5 (Pin_5); no longer J1.2 (Pin_2)
- net IN2: now also J1.3 (Pin_3); no longer J1.4 (Pin_4)
- net IN3: now also J1.1 (Pin_1); no longer J1.6 (Pin_6)
- net SLC1: now also J1.4 (Pin_4); no longer J1.3 (Pin_3)
- net SLS1: now also J1.6 (Pin_6); no longer J1.1 (Pin_1)
Other:
- title: (none) -> End Of Line Testing Board
